Commit message: The Version with dedicated wheels

File: urdf/yahboomcar_X3plus.urdf (robot description, URDF)
Before this commit: robot yahboomcar_X3plus, 17 links, 16 joints
Links:
- removed link arm_link1
- removed link arm_link2
- removed link arm_link3
- removed link arm_link4
- removed link arm_link5
- removed link base_link
- removed link camera_link
- removed link imu_link
- removed link laser_link
- removed link llink1
- removed link llink2
- removed link llink3
- removed link mono_link
- removed link rlink1
- removed link rlink2
- removed link rlink3
Joints:
- removed joint arm_joint1
- removed joint arm_joint2
- removed joint arm_joint3
- removed joint arm_joint4
- removed joint arm_joint5
- removed joint astra_joint
- removed joint base_imu
- removed joint base_joint
- removed joint grip_joint
- removed joint laser_joint
- removed joint llink_joint1
- removed joint llink_joint2
- removed joint llink_joint3
- removed joint mono_joint
- removed joint rlink_joint2
- removed joint rlink_joint3

File: urdf/yahboomcar_X3plus.urdf.xacro (robot description, xacro)
@@ -1,4 +1,4 @@
 <?xml version="1.0" encoding="utf-8"?>
-<robot name="yahboomcar_X3plus" xmlns:xacro="http://wiki.ros.org/xacro">
+<robot name="yahboomcar_X3plus" xmlns:xacro="http://wiki.ros.org/xacro" xmlns:gz="http://gazebosim.org/schema">
   <!-- define the list of relevant args -->
   <!-- <xacro:if value="${namespace == 'None'}">
@@ -15,4 +15,5 @@
     </material>
     <xacro:property name="ns" value="$(arg ns)"/>
+    <xacro:property name="wheel_radius" value="0.05" />
     <link name="base_footprint"/>
     <link name="base_link">
@@ -31,5 +32,5 @@
             <origin xyz="0 0 0" rpy="0 0 0" />
             <geometry>
-                    <mesh filename="package://x3plus_description/meshes/X3plus/visual/base_link.STL"/>
+                    <mesh filename="package://x3plus_description/meshes/X3plus/visual/base-link-core.STL"/>
             </geometry>
             <material name="">
@@ -40,5 +41,5 @@
             <origin xyz="0 0 0" rpy="0 0 0" />
             <geometry>
-                    <mesh filename="package://x3plus_description/meshes/X3plus/collision/base_link.STL"/>
+                    <mesh filename="package://x3plus_description/meshes/X3plus/collision/base-link-core.STL"/>
             </geometry>
         </collision>
@@ -97,4 +98,52 @@
         </joint>
     </xacro:macro>
+      <!-- common mecanum wheel link-->
+    <xacro:macro name="common_mecanum_wheel_link" params="name material fdir *origin">
+        <link name="${name}">
+            <visual>
+                <geometry>
+                    <mesh filename="package://x3plus_description/meshes/X3plus/visual/${name}.STL" />
+                </geometry>
+                <origin xyz="0 0 0" rpy="0 0 0" />
+                <material name="${material}" />
+            </visual>
+            <collision>
+                <pose>0 0 0 0 0 0</pose>
+                <geometry>
+                    <sphere radius="0.032391999999999997" />
+                </geometry>
+            </collision>
+            <xacro:insert_block name="origin" />
+        </link>
+        <gazebo reference="${name}">
+            <collision>
+                <surface>
+                    <contact>
+                        <ode />
+                      </contact>
+                  <friction>
+                    <ode>
+                      <mu>1.0</mu>
+                      <mu2>0.0</mu2>
+                      <fdir1 gz:expressed_in="base_footprint">${fdir}</fdir1>
+                    </ode>
+                  </friction>
+                </surface>
+              </collision>
+            <!-- <mu1>1</mu1>
+            <mu2>0</mu2>
+            <fdir1 gz:expressed_in='base_footprint'>${fdir}</fdir1> -->
+        </gazebo>
+    </xacro:macro>
+    <!-- continuous joint-->
+    <xacro:macro name="wheel_continuous_joint" params="name parent child xyz rpy axis">
+        <joint name="${name}" type="continuous">
+            <parent link="${parent}" />
+            <child link="${child}" />
+            <origin xyz="${xyz}" rpy="${rpy}" />
+            <axis xyz="${axis}" />
+            <limit lower="${-pi}" upper="${pi}" effort="100" velocity="5" />
+        </joint>
+    </xacro:macro>
     <!-- <common_link name="base_link" material="Green" path="X3plus">
         <inertial>
@@ -293,3 +342,47 @@
     <xacro:fixed_joint name="mono_joint" parent="arm_link4" child="mono_link" xyz="-0.0481 -0.05145 -0.0022"
                  rpy="${pi/2} 0 0"/>
+   <xacro:common_mecanum_wheel_link name="front_right_wheel" material="White" fdir="1 1 0">
+            <inertial>
+                <origin xyz="1.9051E-06 -2.3183E-07 -0.00064079" rpy="0 0 0" />
+                <mass value="0.051532" />
+                <inertia ixx="1.4595E-05" ixy="-4.3975E-10" ixz="4.415E-10"
+                    iyy="1.4594E-05" iyz="-1.7476E-09" izz="2.4264E-05" />
+            </inertial>
+        </xacro:common_mecanum_wheel_link>
+        <xacro:common_mecanum_wheel_link name="front_left_wheel" material="White" fdir="1 -1 0">
+            <inertial>
+                <origin xyz="2.3728E-06 -9.4228E-07 0.00064068" rpy="0 0 0" />
+                <mass value="0.051543" />
+                <inertia ixx="1.4597E-05" ixy="-4.7945E-10" ixz="-2.4786E-10"
+                    iyy="1.4598E-05" iyz="1.7972E-09" izz="2.4267E-05" />
+            </inertial>
+        </xacro:common_mecanum_wheel_link>
+        <xacro:common_mecanum_wheel_link name="back_right_wheel" material="White" fdir="1 -1 0">
+            <inertial>
+                <origin xyz="-1.75924169923403E-06 1.28388821071107E-06 -0.000590549296238266"
+                    rpy="0 0 0" />
+                <mass value="0.051540174053366" />
+                <inertia ixx="1.45974152250002E-05" ixy="1.94850559178397E-10"
+                    ixz="-1.61846387282284E-09"
+                    iyy="1.4596501955693E-05" iyz="-6.27904057423818E-10" izz="2.42663091380451E-05" />
+            </inertial>
+        </xacro:common_mecanum_wheel_link>
+        <xacro:common_mecanum_wheel_link name="back_left_wheel" material="White" fdir="1 1 0">
+            <inertial>
+                <origin xyz="-4.01213085227115E-07 2.04910264598596E-06 0.000590775697051377"
+                    rpy="0 0 0" />
+                <mass value="0.0515309299357028" />
+                <inertia ixx="1.45942986129926E-05" ixy="-3.19787215398093E-10"
+                    ixz="1.74943062058915E-09"
+                    iyy="1.45948727598913E-05" iyz="1.61769812110049E-10" izz="2.4263683888153E-05" />
+            </inertial>
+        </xacro:common_mecanum_wheel_link>
+    <xacro:wheel_continuous_joint name="front_right_joint" parent="base_link" child="front_right_wheel"
+        xyz="0.105  -0.103 -0.038" rpy="${pi/2} 0 ${pi}" axis="0 0 1" />
+    <xacro:wheel_continuous_joint name="front_left_joint" parent="base_link" child="front_left_wheel"
+        xyz="0.105   0.103 -0.038" rpy="${pi/2} 0 0" axis="0 0 1" />
+    <xacro:wheel_continuous_joint name="back_right_joint" parent="base_link" child="back_right_wheel"
+        xyz="-0.115 -0.103 -0.038" rpy="${pi/2} 0 ${pi}" axis="0 0 1" />
+    <xacro:wheel_continuous_joint name="back_left_joint" parent="base_link" child="back_left_wheel"
+        xyz="-0.115  0.103 -0.038" rpy="${pi/2} 0 0" axis="0 0 1" />
 </robot>
