Commit message: Working on the X3plus

File: urdf/yahboomcar_X3plusX.urdf.xacro (robot description, xacro)
@@ -1,6 +1,7 @@
 <?xml version="1.0" encoding="utf-8"?>
-<robot name="yahboomcar_X3plus" xmlns:xacro="http://wiki.ros.org/xacro" xmlns:gz="http://gazebosim.org/schema">
-  <!-- define the list of relevant args -->
-  <!-- <xacro:if value="${namespace == 'None'}">
+<robot name="yahboomcar_X3plus" xmlns:xacro="http://wiki.ros.org/xacro"
+    xmlns:gz="http://gazebosim.org/schema">
+    <!-- define the list of relevant args -->
+    <!-- <xacro:if value="${namespace == 'None'}">
         <xacro:property name="ns" value="" />
       </xacro:if>
@@ -9,28 +10,29 @@
       </xacro:unless> -->
     <material name="Green">
-        <color rgba="0 0.7 0 1"/>
+        <color rgba="0 0.7 0 1" />
     </material>
     <material name="White">
-        <color rgba="0.7 0.7 0.7 1"/>
+        <color rgba="0.7 0.7 0.7 1" />
     </material>
-    <xacro:property name="ns" value="$(arg ns)"/>
+    <xacro:property name="ns" value="$(arg ns)" />
     <xacro:property name="wheel_radius" value="0.05" />
-    <link name="base_footprint"/>
+    <link name="base_footprint" />
     <link name="base_link">
         <inertial>
-            <origin xyz="-0.0304416859098744 4.23384368655101E-05 0.0448234503408059" rpy="0 0 0"/>
-            <mass value="1.0754239466482"/>
-            <inertia
-                    ixx="0.0208831789264125"
-                    ixy="2.4618093127858E-06"
-                    ixz="0.00616019290028669"
-                    iyy="0.0265621377486244"
-                    iyz="-1.10079499865282E-06"
-                    izz="0.0129535610833954"/>
+            <origin xyz="-0.0304416859098744 4.23384368655101E-05 0.0448234503408059" rpy="0 0 0" />
+            <mass value="1.0754239466482" />
+            <inertia
+                ixx="0.0208831789264125"
+                ixy="2.4618093127858E-06"
+                ixz="0.00616019290028669"
+                iyy="0.0265621377486244"
+                iyz="-1.10079499865282E-06"
+                izz="0.0129535610833954" />
         </inertial>
         <visual>
             <origin xyz="0 0 0" rpy="0 0 0" />
             <geometry>
-                    <mesh filename="package://x3plus_description/meshes/X3plus/visual/base-link-small.STL"/>
+                <mesh
+                    filename="package://x3plus_description/meshes/X3plus/visual/base-link-small.STL" />
             </geometry>
             <material name="">
@@ -41,5 +43,6 @@
             <origin xyz="0 0 0" rpy="0 0 0" />
             <geometry>
-                    <mesh filename="package://x3plus_description/meshes/X3plus/collision/base-link-small.STL"/>
+                <mesh
+                    filename="package://x3plus_description/meshes/X3plus/collision/base-link-small.STL" />
             </geometry>
         </collision>
@@ -56,16 +59,17 @@
             <visual>
                 <geometry>
-                    <mesh filename="package://x3plus_description/meshes/${path}/visual/${name}.STL"/>
+                    <mesh filename="package://x3plus_description/meshes/${path}/visual/${name}.STL" />
                 </geometry>
-                <origin xyz="0 0 0" rpy="0 0 0"/>
-                <material name="${material}"/>
+                <origin xyz="0 0 0" rpy="0 0 0" />
+                <material name="${material}" />
             </visual>
             <collision>
                 <geometry>
-                    <mesh filename="package://x3plus_description/meshes/${path}/collision/${name}.STL"/>
+                    <mesh
+                        filename="package://x3plus_description/meshes/${path}/collision/${name}.STL" />
                 </geometry>
-                <origin xyz="0 0 0" rpy="0 0 0"/>
+                <origin xyz="0 0 0" rpy="0 0 0" />
             </collision>
-            <xacro:insert_block name="origin"/>
+            <xacro:insert_block name="origin" />
         </link>
     </xacro:macro>
@@ -73,9 +77,9 @@
     <xacro:macro name="revolute_joint" params="name parent child xyz rpy axisZ lower upper">
         <joint name="${name}" type="revolute">
-            <parent link="${parent}"/>
-            <child link="${child}"/>
-            <origin xyz="${xyz}" rpy="${rpy}"/>
-            <axis xyz="0 0 ${axisZ}"/>
-            <limit lower="${lower}" upper="${upper}" effort="100" velocity="1"/>
+            <parent link="${parent}" />
+            <child link="${child}" />
+            <origin xyz="${xyz}" rpy="${rpy}" />
+            <axis xyz="0 0 ${axisZ}" />
+            <limit lower="${lower}" upper="${upper}" effort="100" velocity="1" />
         </joint>
     </xacro:macro>
@@ -83,9 +87,9 @@
     <xacro:macro name="continuous_joint" params="name parent child xyz rpy mimic">
         <joint name="${name}" type="continuous">
-            <parent link="${parent}"/>
-            <child link="${child}"/>
-            <origin xyz="${xyz}" rpy="${rpy}"/>
-            <axis xyz="0 0 1"/>
-            <mimic joint="grip_joint" multiplier="${mimic}"/>
+            <parent link="${parent}" />
+            <child link="${child}" />
+            <origin xyz="${xyz}" rpy="${rpy}" />
+            <axis xyz="0 0 1" />
+            <mimic joint="grip_joint" multiplier="${mimic}" />
         </joint>
     </xacro:macro>
@@ -93,10 +97,10 @@
     <xacro:macro name="fixed_joint" params="name parent child xyz rpy">
         <joint name="${name}" type="fixed">
-            <parent link="${parent}"/>
-            <child link="${child}"/>
-            <origin xyz="${xyz}" rpy="${rpy}"/>
+            <parent link="${parent}" />
+            <child link="${child}" />
+            <origin xyz="${xyz}" rpy="${rpy}" />
         </joint>
     </xacro:macro>
-      <!-- common mecanum wheel link-->
+    <!-- common mecanum wheel link-->
     <xacro:macro name="common_mecanum_wheel_link" params="name material fdir *origin">
         <link name="${name}">
@@ -121,14 +125,14 @@
                     <contact>
                         <ode />
-                      </contact>
-                  <friction>
-                    <ode>
-                      <mu>1.0</mu>
-                      <mu2>0.0</mu2>
-                      <fdir1 gz:expressed_in="base_footprint">${fdir}</fdir1>
-                    </ode>
-                  </friction>
+                    </contact>
+                    <friction>
+                        <ode>
+                            <mu>1.0</mu>
+                            <mu2>0.0</mu2>
+                            <fdir1 gz:expressed_in="base_footprint">${fdir}</fdir1>
+                        </ode>
+                    </friction>
                 </surface>
-              </collision>
+            </collision>
             <!-- <mu1>1</mu1>
             <mu2>0</mu2>
@@ -159,53 +163,67 @@
         </inertial>
     </common_link>
-    <fixed_joint name="base_joint" parent="base_footprint" child="base_link" xyz="0.0 0.0 0.076" rpy="0 0 0"/> -->
-    <!-- <fixed_joint name="base_imu" parent="base_link" child="imu_link" xyz="0.001 0.017 0.0322" rpy="0 3.1415 1.5707"/> -->
+    <fixed_joint name="base_joint" parent="base_footprint" child="base_link" xyz="0.0 0.0 0.076" rpy="0
+    0 0"/> -->
+    <!-- <fixed_joint name="base_imu" parent="base_link" child="imu_link" xyz="0.001 0.017 0.0322"
+    rpy="0 3.1415 1.5707"/> -->
     <xacro:common_link name="laser_link" material="White" path="sensor">
         <inertial>
-            <origin xyz="-0.0176558922685589 0.000671805271544437 0.0219302095894866" rpy="0 0 0"/>
-            <mass value="0.0483909504209895"/>
-            <inertia ixx="1.58456966399128E-05" ixy="-4.23913983850005E-07" ixz="-2.09597897904374E-07"
-                     iyy="3.89262522903605E-05" iyz="3.24809725932687E-07" izz="4.86230801106223E-05"/>
-        </inertial>
-    </xacro:common_link>
-    <xacro:fixed_joint name="laser_joint" parent="base_link" child="laser_link" xyz="0.10478 0 0.0471" rpy="0 0 0"/>
+            <origin xyz="-0.0176558922685589 0.000671805271544437 0.0219302095894866" rpy="0 0 0" />
+            <mass value="0.0483909504209895" />
+            <inertia ixx="1.58456966399128E-05" ixy="-4.23913983850005E-07"
+                ixz="-2.09597897904374E-07"
+                iyy="3.89262522903605E-05" iyz="3.24809725932687E-07" izz="4.86230801106223E-05" />
+        </inertial>
+    </xacro:common_link>
+    <xacro:fixed_joint name="laser_joint" parent="base_link" child="laser_link"
+        xyz="0.10478 0 0.0471" rpy="0 0 0" />
     <xacro:common_link name="camera_link" material="White" path="sensor">
         <inertial>
-            <origin xyz="0 0 0" rpy="0 0 0"/>
-            <mass value="0"/>
-            <inertia ixx="0" ixy="0" ixz="0" iyy="0" iyz="0" izz="0"/>
-        </inertial>
-    </xacro:common_link>
+            <origin xyz="0 0 0" rpy="0 0 0" />
+            <mass value="0" />
+            <inertia ixx="0" ixy="0" ixz="0" iyy="0" iyz="0" izz="0" />
+        </inertial>
+    </xacro:common_link>
+    <xacro:fixed_joint name="camera_joint" parent="base_link" child="camera_link"
+        xyz="0.057105 1.7948E-05 0.03755" rpy="0 0 0" />
+   <joint name="camera_optical_joint" type="fixed">
+            <origin xyz="0 0 0" rpy="${-pi/2} 0 ${-pi/2}" />
+            <parent link="camera_link" />
+            <child link="camera_link_optical" />
+        </joint>
+        <link name="camera_link_optical"></link>
     <xacro:common_link name="arm_link1" material="White" path="X3plus">
         <inertial>
-            <origin xyz="1.99179507982521E-05 -5.98354652829568E-05 0.0114289358828097" rpy="0 0 0"/>
-            <mass value="0.0279545499871709"/>
-            <inertia
-                    ixx="1.19144359314975E-05"
-                    ixy="-9.26068510046816E-09"
-                    ixz="3.16060516198683E-09"
-                    iyy="1.05642517915377E-05"
-                    iyz="2.69674403668579E-08"
-                    izz="1.49639510661413E-05"/>
-        </inertial>
-    </xacro:common_link>
-    <xacro:revolute_joint name="arm_joint1" parent="base_link" child="arm_link1" xyz="0.09825 0 0.102" rpy="0 0 0" axisZ="-1"
-                    lower="-${pi/2}" upper="${pi/2}"/>
+            <origin xyz="1.99179507982521E-05 -5.98354652829568E-05 0.0114289358828097" rpy="0 0 0" />
+            <mass value="0.0279545499871709" />
+            <inertia
+                ixx="1.19144359314975E-05"
+                ixy="-9.26068510046816E-09"
+                ixz="3.16060516198683E-09"
+                iyy="1.05642517915377E-05"
+                iyz="2.69674403668579E-08"
+                izz="1.49639510661413E-05" />
+        </inertial>
+    </xacro:common_link>
+    <xacro:revolute_joint name="arm_joint1" parent="base_link" child="arm_link1"
+        xyz="0.09825 0 0.102" rpy="0 0 0" axisZ="-1"
+        lower="-${pi/2}" upper="${pi/2}" />
     <xacro:common_link name="arm_link2b" material="Green" path="X3plus">
         <inertial>
-            <origin xyz="0.024903 -0.0022632 -0.00066663" rpy="0 0 0"/>
-            <mass value="0.031605"/>
-            <inertia
-                    ixx="5.8495E-06"
-                    ixy="-8.8092E-07"
-                    ixz="1.5336E-07"
-                    iyy="2.667E-05"
-                    iyz="7.1365E-09"
-                    izz="2.4695E-05"/>
+            <origin xyz="0.024903 -0.0022632 -0.00066663" rpy="0 0 0" />
+            <mass value="0.031605" />
+            <inertia
+                ixx="5.8495E-06"
+                ixy="-8.8092E-07"
+                ixz="1.5336E-07"
+                iyy="2.667E-05"
+                iyz="7.1365E-09"
+                izz="2.4695E-05" />
         </inertial>
     </xacro:common_link>
     <xacro:revolute_joint name="arm_joint2" parent="arm_link1" child="arm_link2b" xyz="0 0 0.0405"
-                    rpy="-${pi/2} 0 0" axisZ="-1" lower="-${pi/2}" upper="${pi/2}"/>
-    <xacro:fixed_joint name="camera_joint" parent="arm_link2b" child="camera_link" xyz="0 -0.07 0" rpy="${pi/2} 0 0"/>
+        rpy="-${pi/2} 0 0" axisZ="-1" lower="-${pi/2}" upper="${pi/2}" />
+    <xacro:fixed_joint name="camera_joint" parent="arm_link2b" child="camera_link" xyz="0 -0.07 0"
+        rpy="${pi/2} 0 0" />
     <!-- <xacro:common_link name="arm_link3" material="White" path="X3plus">
         <inertial>
@@ -221,5 +239,6 @@
         </inertial>
     </xacro:common_link>
-    <xacro:revolute_joint name="arm_joint3" parent="arm_link2" child="arm_link3" xyz="0 -0.0829 0" rpy="0 0 0"
+    <xacro:revolute_joint name="arm_joint3" parent="arm_link2" child="arm_link3" xyz="0 -0.0829 0"
+    rpy="0 0 0"
                     axisZ="-1" lower="-${pi/2}" upper="${pi/2}"/>
     <xacro:common_link name="arm_link4" material="Green" path="X3plus">
@@ -236,5 +255,6 @@
         </inertial>
     </xacro:common_link>
-    <xacro:revolute_joint name="arm_joint4" parent="arm_link3" child="arm_link4" xyz="0 -0.0829 0" rpy="0 0 0"
+    <xacro:revolute_joint name="arm_joint4" parent="arm_link3" child="arm_link4" xyz="0 -0.0829 0"
+    rpy="0 0 0"
                     axisZ="-1" lower="-${pi/2}" upper="${pi/2}"/>
     <xacro:common_link name="arm_link5" material="White" path="X3plus">
@@ -251,5 +271,6 @@
         </inertial>
     </xacro:common_link>
-    <xacro:revolute_joint name="arm_joint5" parent="arm_link4" child="arm_link5" xyz="-0.00215 -0.17455 0"
+    <xacro:revolute_joint name="arm_joint5" parent="arm_link4" child="arm_link5" xyz="-0.00215 -0.17455
+    0"
                     rpy="${pi/2} 0 0" axisZ="1" lower="-${pi/2}" upper="${pi}"/>
     <xacro:common_link name="rlink1" material="Green" path="X3plus">
@@ -266,5 +287,6 @@
         </inertial>
     </xacro:common_link>
-    <xacro:revolute_joint name="grip_joint" parent="arm_link5" child="rlink1" xyz="-0.0035 -0.012625 -0.0685"
+    <xacro:revolute_joint name="grip_joint" parent="arm_link5" child="rlink1" xyz="-0.0035 -0.012625
+    -0.0685"
                     rpy="0 -${pi/2} 0" axisZ="1" lower="-${pi/2}" upper="0"/>
     <xacro:common_link name="rlink2" material="Green" path="X3plus">
@@ -281,5 +303,6 @@
         </inertial>
     </xacro:common_link>
-    <xacro:continuous_joint name="rlink_joint2" parent="rlink1" child="rlink2" xyz="0.03 -0.00075429 0" rpy="0 0 0" mimic="-1"/>
+    <xacro:continuous_joint name="rlink_joint2" parent="rlink1" child="rlink2" xyz="0.03 -0.00075429 0"
+    rpy="0 0 0" mimic="-1"/>
     <xacro:common_link name="rlink3" material="Green" path="X3plus">
         <inertial>
@@ -295,5 +318,6 @@
         </inertial>
     </xacro:common_link>
-    <xacro:continuous_joint name="rlink_joint3" parent="arm_link5" child="rlink3" xyz="-0.0035 -0.0045 -0.0505"
+    <xacro:continuous_joint name="rlink_joint3" parent="arm_link5" child="rlink3" xyz="-0.0035 -0.0045
+    -0.0505"
                       rpy="0 -${pi/2} 0" mimic="1"/>
     <xacro:common_link name="llink1" material="Green" path="X3plus">
@@ -310,5 +334,6 @@
         </inertial>
     </xacro:common_link>
-    <xacro:continuous_joint name="llink_joint1" parent="arm_link5" child="llink1" xyz="-0.0035 0.012375 -0.0685"
+    <xacro:continuous_joint name="llink_joint1" parent="arm_link5" child="llink1" xyz="-0.0035 0.012375
+    -0.0685"
                       rpy="0 -${pi/2} 0" mimic="-1"/>
     <xacro:common_link name="llink2" material="Green" path="X3plus">
@@ -320,5 +345,6 @@
         </inertial>
     </xacro:common_link>
-    <xacro:continuous_joint name="llink_joint2" parent="llink1" child="llink2" xyz="0.03 0.00065104 0" rpy="0 0 0"
+    <xacro:continuous_joint name="llink_joint2" parent="llink1" child="llink2" xyz="0.03 0.00065104 0"
+    rpy="0 0 0"
                       mimic="1"/>
     <xacro:common_link name="llink3" material="Green" path="X3plus">
@@ -330,5 +356,6 @@
         </inertial>
     </xacro:common_link>
-    <xacro:continuous_joint name="llink_joint3" parent="arm_link5" child="llink3" xyz="-0.0035 0.0045 -0.0505"
+    <xacro:continuous_joint name="llink_joint3" parent="arm_link5" child="llink3" xyz="-0.0035 0.0045
+    -0.0505"
                       rpy="0 -${pi/2} 0" mimic="-1"/>
     <xacro:common_link name="mono_link" material="White" path="sensor">
@@ -340,50 +367,324 @@
         </inertial>
     </xacro:common_link>
-    <xacro:fixed_joint name="mono_joint" parent="arm_link4" child="mono_link" xyz="-0.0481 -0.05145 -0.0022"
+    <xacro:fixed_joint name="mono_joint" parent="arm_link4" child="mono_link" xyz="-0.0481 -0.05145
+    -0.0022"
                  rpy="${pi/2} 0 0"/>
                  -->
-   <xacro:common_mecanum_wheel_link name="front_right_wheel" material="White" fdir="1 1 0">
-            <inertial>
-                <origin xyz="1.9051E-06 -2.3183E-07 -0.00064079" rpy="0 0 0" />
-                <mass value="0.051532" />
-                <inertia ixx="1.4595E-05" ixy="-4.3975E-10" ixz="4.415E-10"
-                    iyy="1.4594E-05" iyz="-1.7476E-09" izz="2.4264E-05" />
-            </inertial>
-        </xacro:common_mecanum_wheel_link>
-        <xacro:common_mecanum_wheel_link name="front_left_wheel" material="White" fdir="1 -1 0">
-            <inertial>
-                <origin xyz="2.3728E-06 -9.4228E-07 0.00064068" rpy="0 0 0" />
-                <mass value="0.051543" />
-                <inertia ixx="1.4597E-05" ixy="-4.7945E-10" ixz="-2.4786E-10"
-                    iyy="1.4598E-05" iyz="1.7972E-09" izz="2.4267E-05" />
-            </inertial>
-        </xacro:common_mecanum_wheel_link>
-        <xacro:common_mecanum_wheel_link name="back_right_wheel" material="White" fdir="1 -1 0">
-            <inertial>
-                <origin xyz="-1.75924169923403E-06 1.28388821071107E-06 -0.000590549296238266"
-                    rpy="0 0 0" />
-                <mass value="0.051540174053366" />
-                <inertia ixx="1.45974152250002E-05" ixy="1.94850559178397E-10"
-                    ixz="-1.61846387282284E-09"
-                    iyy="1.4596501955693E-05" iyz="-6.27904057423818E-10" izz="2.42663091380451E-05" />
-            </inertial>
-        </xacro:common_mecanum_wheel_link>
-        <xacro:common_mecanum_wheel_link name="back_left_wheel" material="White" fdir="1 1 0">
-            <inertial>
-                <origin xyz="-4.01213085227115E-07 2.04910264598596E-06 0.000590775697051377"
-                    rpy="0 0 0" />
-                <mass value="0.0515309299357028" />
-                <inertia ixx="1.45942986129926E-05" ixy="-3.19787215398093E-10"
-                    ixz="1.74943062058915E-09"
-                    iyy="1.45948727598913E-05" iyz="1.61769812110049E-10" izz="2.4263683888153E-05" />
-            </inertial>
-        </xacro:common_mecanum_wheel_link>
-    <xacro:wheel_continuous_joint name="front_right_joint" parent="base_link" child="front_right_wheel"
+    <xacro:common_mecanum_wheel_link name="front_right_wheel" material="White" fdir="1 1 0">
+        <inertial>
+            <origin xyz="1.9051E-06 -2.3183E-07 -0.00064079" rpy="0 0 0" />
+            <mass value="0.051532" />
+            <inertia ixx="1.4595E-05" ixy="-4.3975E-10" ixz="4.415E-10"
+                iyy="1.4594E-05" iyz="-1.7476E-09" izz="2.4264E-05" />
+        </inertial>
+    </xacro:common_mecanum_wheel_link>
+    <xacro:common_mecanum_wheel_link name="front_left_wheel" material="White" fdir="1 -1 0">
+        <inertial>
+            <origin xyz="2.3728E-06 -9.4228E-07 0.00064068" rpy="0 0 0" />
+            <mass value="0.051543" />
+            <inertia ixx="1.4597E-05" ixy="-4.7945E-10" ixz="-2.4786E-10"
+                iyy="1.4598E-05" iyz="1.7972E-09" izz="2.4267E-05" />
+        </inertial>
+    </xacro:common_mecanum_wheel_link>
+    <xacro:common_mecanum_wheel_link name="back_right_wheel" material="White" fdir="1 -1 0">
+        <inertial>
+            <origin xyz="-1.75924169923403E-06 1.28388821071107E-06 -0.000590549296238266"
+                rpy="0 0 0" />
+            <mass value="0.051540174053366" />
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