Commit message: fixing camera link

File: urdf/yahboomcar_X3plusX.urdf.xacro (robot description, xacro)
@@ -185,6 +185,39 @@
         </inertial>
     </xacro:common_link>
-    <xacro:fixed_joint name="camera_joint" parent="base_link" child="camera_link"
-        xyz="0.057105 1.7948E-05 0.03755" rpy="0 0 0" />
+    <xacro:common_link name="arm_link1" material="White" path="X3plus">
+        <inertial>
+            <origin xyz="1.99179507982521E-05 -5.98354652829568E-05 0.0114289358828097" rpy="0 0 0" />
+            <mass value="0.0279545499871709" />
+            <inertia
+                ixx="1.19144359314975E-05"
+                ixy="-9.26068510046816E-09"
+                ixz="3.16060516198683E-09"
+                iyy="1.05642517915377E-05"
+                iyz="2.69674403668579E-08"
+                izz="1.49639510661413E-05" />
+        </inertial>
+    </xacro:common_link>
+    <xacro:revolute_joint name="arm_joint1" parent="base_link" child="arm_link1"
+        xyz="0.09825 0 0.102" rpy="0 0 0" axisZ="-1"
+        lower="-${pi/2}" upper="${pi/2}" />
+    <xacro:common_link name="arm_link2b" material="Green" path="X3plus">
+        <inertial>
+            <origin xyz="0.024903 -0.0022632 -0.00066663" rpy="0 0 0" />
+            <mass value="0.031605" />
+            <inertia
+                ixx="5.8495E-06"
+                ixy="-8.8092E-07"
+                ixz="1.5336E-07"
+                iyy="2.667E-05"
+                iyz="7.1365E-09"
+                izz="2.4695E-05" />
+        </inertial>
+    </xacro:common_link>
+    <xacro:revolute_joint name="arm_joint2" parent="arm_link1" child="arm_link2b" xyz="0 0 0.0405"
+        rpy="-${pi/2} 0 0" axisZ="-1" lower="-${pi/2}" upper="${pi/2}" />
+    <xacro:fixed_joint name="camera_joint" parent="arm_link2b" child="camera_link" xyz="0 -0.07 0"
+        rpy="${pi/2} 0 0" />
+    <!-- <xacro:fixed_joint name="camera_joint" parent="base_link" child="camera_link"
+        xyz="0.057105 1.7948E-05 0.03755" rpy="0 0 0" /> -->
    <joint name="camera_optical_joint" type="fixed">
             <origin xyz="0 0 0" rpy="${-pi/2} 0 ${-pi/2}" />
@@ -193,37 +226,4 @@
         </joint>
         <link name="camera_link_optical"></link>
-    <xacro:common_link name="arm_link1" material="White" path="X3plus">
-        <inertial>
-            <origin xyz="1.99179507982521E-05 -5.98354652829568E-05 0.0114289358828097" rpy="0 0 0" />
-            <mass value="0.0279545499871709" />
-            <inertia
-                ixx="1.19144359314975E-05"
-                ixy="-9.26068510046816E-09"
-                ixz="3.16060516198683E-09"
-                iyy="1.05642517915377E-05"
-                iyz="2.69674403668579E-08"
-                izz="1.49639510661413E-05" />
-        </inertial>
-    </xacro:common_link>
-    <xacro:revolute_joint name="arm_joint1" parent="base_link" child="arm_link1"
-        xyz="0.09825 0 0.102" rpy="0 0 0" axisZ="-1"
-        lower="-${pi/2}" upper="${pi/2}" />
-    <xacro:common_link name="arm_link2b" material="Green" path="X3plus">
-        <inertial>
-            <origin xyz="0.024903 -0.0022632 -0.00066663" rpy="0 0 0" />
-            <mass value="0.031605" />
-            <inertia
-                ixx="5.8495E-06"
-                ixy="-8.8092E-07"
-                ixz="1.5336E-07"
-                iyy="2.667E-05"
-                iyz="7.1365E-09"
-                izz="2.4695E-05" />
-        </inertial>
-    </xacro:common_link>
-    <xacro:revolute_joint name="arm_joint2" parent="arm_link1" child="arm_link2b" xyz="0 0 0.0405"
-        rpy="-${pi/2} 0 0" axisZ="-1" lower="-${pi/2}" upper="${pi/2}" />
-    <xacro:fixed_joint name="camera_joint" parent="arm_link2b" child="camera_link" xyz="0 -0.07 0"
-        rpy="${pi/2} 0 0" />
     <!-- <xacro:common_link name="arm_link3" material="White" path="X3plus">
         <inertial>
